File: dynamis.kicad_pcb (KiCad board)
At the start: 2 copper layers, 18.3 x 9.1 mm, 189 parts, among them J0 USB_C_Receptacle_USB2.0, SW00_00 SW_Push, SW00_01 SW_Push, SW00_02 SW_Push, SW00_03 SW_Push, SW00_04 SW_Push, SW00_05 SW_Push, SW00_06 SW_Push, SW01_00 SW_Push, SW01_01 SW_Push, SW01_02 SW_Push, SW01_03 SW_Push, SW01_04 SW_Push, SW01_05 SW_Push, SW01_06 SW_Push, SW02_01 SW_Push, SW02_02 SW_Push, SW02_03 SW_Push, SW02_04 SW_Push, SW02_05 SW_Push, SW02_06 SW_Push, SW03_00 SW_Push, SW03_02 SW_Push, SW03_03 SW_Push, SW03_04 SW_Push, SW03_05 SW_Push, SW03_06 SW_Push, SW04_00 SW_Push, SW04_01 SW_Push, SW04_02 SW_Push, SW04_03 SW_Push, SW04_05 SW_Push, SW04_06 SW_Push, SW05_01 SW_Push, SW05_02 SW_Push, SW05_03 SW_Push, SW05_04 SW_Push, SW05_05 SW_Push, SW05_06 SW_Push, SW06_00 SW_Push, SW06_01 SW_Push, SW06_02 SW_Push, SW06_03 SW_Push, SW06_04 SW_Push, SW06_05 SW_Push, SW06_06 SW_Push, SW07_01 SW_Push, SW07_02 SW_Push, SW07_03 SW_Push, SW07_04 SW_Push, SW07_05 SW_Push, SW07_06 SW_Push, SW08_00 SW_Push, SW08_02 SW_Push, SW08_03 SW_Push, SW08_04 SW_Push, SW08_05 SW_Push, SW08_06 SW_Push, SW09_00 SW_Push, SW09_01 SW_Push, SW09_02 SW_Push, SW09_03 SW_Push, SW09_04 SW_Push, SW09_05 SW_Push, SW09_06 SW_Push, U0 ATmega32U4-A, U1 PMW3360DM-T2QU, U2 TLV70019DDCR, U3 74LVC1T45GW,125, U4 74LVC1T45GW,125, U5 74LVC1T45GW,125, U6 74LVC1T45GW,125, U7 74LVC1T45GW,125, Y0 16Mhz

Commit message: wip
Parts:
- added AN_STAB_00: 2.25U, MX_Only:MXOnly-2.25U-ReversedStabilizers-NoSwitch, F.Cu at (397.2, 248.9)
- added IS_STAB_00: ISO, MX_Only:MXOnly-ISO-ReversedStabilizers-NoSwitch, F.Cu at (406.7, 239.4)
- added LED5: WS2812B, LED_SMD:LED_WS2812B_PLCC4_5.0x5.0mm_P3.2mm, F.Cu at (532.6, 305.0)
- added LED6: WS2812B, LED_SMD:LED_WS2812B_PLCC4_5.0x5.0mm_P3.2mm, F.Cu at (541.1, 305.0)
- SW01_00: footprint MX_Only:MXOnly-1U-Hotswap -> MX_Only:MXOnly-1.5U-Hotswap
- SW03_00, SW04_00, SW04_01, SW04_02, SW04_06, SW09_05, SW09_06, SWSP_S04: footprint MX_Only:MXOnly-1U-Hotswap -> MX_Only:MXOnly-1.25U-Hotswap
- SW04_03: footprint MX_Only:MXOnly-1U-Hotswap -> MX_Only:MXOnly-2.25U-Hotswap-ReversedStabilizers
- SW04_05: footprint MX_Only:MXOnly-1U-Hotswap -> MX_Only:MXOnly-2.75U-Hotswap-ReversedStabilizers
- SWBS_L00: footprint MX_Only:MXOnly-1U-Hotswap -> MX_Only:MXOnly-2U-Hotswap
- SWCL_N00, SWRS_S01: footprint MX_Only:MXOnly-1U-Hotswap -> MX_Only:MXOnly-1.75U-Hotswap
- SWLS_L01: footprint MX_Only:MXOnly-1U-Hotswap -> MX_Only:MXOnly-2.25U-Hotswap
- SWRS_L01: footprint MX_Only:MXOnly-1U-Hotswap -> MX_Only:MXOnly-2.75U-Hotswap
- SWSP_L04: footprint MX_Only:MXOnly-1U-Hotswap -> MX_Only:MXOnly-6.25U-Hotswap
- moved SW09_03 422.0 mm to (432.9, 287.0)
- moved SW08_00 419.6 mm to (409.1, 268.0), turned to 180 degrees
- moved SW09_06 394.3 mm to (359.1, 287.0)
- moved SW09_01 385.4 mm to (432.9, 268.0)
- moved SWET_IS00 385.3 mm to (406.7, 239.4), turned to 90 degrees
- moved LED1 379.7 mm to (526.8, 251.2)
- moved SW04_06 363.2 mm to (335.3, 287.0)
- moved SWRS_L01 358.5 mm to (392.4, 268.0)
- moved SW06_01 346.7 mm to (380.5, 229.9)
- moved SW07_05 343.5 mm to (309.1, 248.9)
- moved SW09_02 340.6 mm to (451.9, 287.0)
- moved C0 330.4 mm to (530.0, 281.1)
- moved C4 330.4 mm to (489.6, 321.6)
- moved C8 330.4 mm to (520.8, 288.1)
- moved C9 330.4 mm to (475.3, 335.2)
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- renumbered LED8 to LED10, LED9 to LED11, LED5 to LED7, LED6 to LED8, LED7 to LED9
Connections:
- LED7 pad 4: Net-(LED4-Pad2) -> Net-(LED7-Pad4)
