File: dynamis.kicad_pcb (KiCad board)
At the start: 2 copper layers, 18.3 x 9.1 mm, 249 parts, among them J0 USB_C_Receptacle_USB2.0, SW00_00 SW_Push, SW00_01 SW_Push, SW00_02 SW_Push, SW00_03 SW_Push, SW00_04 SW_Push, SW00_05 SW_Push, SW00_06 SW_Push, SW01_00 SW_Push, SW01_01 SW_Push, SW01_02 SW_Push, SW01_03 SW_Push, SW01_04 SW_Push, SW01_05 SW_Push, SW01_06 SW_Push, SW02_01 SW_Push, SW02_02 SW_Push, SW02_03 SW_Push, SW02_04 SW_Push, SW02_05 SW_Push, SW02_06 SW_Push, SW03_00 SW_Push, SW03_02 SW_Push, SW03_03 SW_Push, SW03_04 SW_Push, SW03_05 SW_Push, SW03_06 SW_Push, SW04_00 SW_Push, SW04_01 SW_Push, SW04_02 SW_Push, SW04_03 SW_Push, SW04_05 SW_Push, SW04_06 SW_Push, SW05_01 SW_Push, SW05_02 SW_Push, SW05_03 SW_Push, SW05_04 SW_Push, SW05_05 SW_Push, SW05_06 SW_Push, SW06_00 SW_Push, SW06_01 SW_Push, SW06_02 SW_Push, SW06_03 SW_Push, SW06_04 SW_Push, SW06_05 SW_Push, SW06_06 SW_Push, SW07_01 SW_Push, SW07_02 SW_Push, SW07_03 SW_Push, SW07_04 SW_Push, SW07_05 SW_Push, SW07_06 SW_Push, SW08_00 SW_Push, SW08_02 SW_Push, SW08_03 SW_Push, SW08_04 SW_Push, SW08_05 SW_Push, SW08_06 SW_Push, SW09_00 SW_Push, SW09_01 SW_Push, SW09_02 SW_Push, SW09_03 SW_Push, SW09_04 SW_Push, SW09_05 SW_Push, SW09_06 SW_Push, U0 ATmega32U4-A, U1 PMW3360DM-T2QU, U2 TLV70019DDCR, U3 74LVC1T45GW,125, U4 74LVC1T45GW,125, U5 74LVC1T45GW,125, U6 74LVC1T45GW,125, U7 74LVC1T45GW,125, Y0 16Mhz

Commit message: wip
Parts:
- removed C0, C1: 22pF, Capacitor_SMD:C_1206_3216Metric
- removed C10: 10μF, Capacitor_SMD:C_1206_3216Metric
- removed C2, C5, C6: 1μF, Capacitor_SMD:C_1206_3216Metric
- removed C3: 4.7μF, Capacitor_SMD:C_1206_3216Metric
- removed C4, C7, C8, C9: 0.1μF, Capacitor_SMD:C_1206_3216Metric
- removed D00_00, D00_01, D00_02, D00_03, D00_04, D00_05, D00_06, D01_00, D01_01, D01_02, D01_03, D01_04, D01_05, D01_06, D02_00, D02_01, D02_02, D02_03, D02_04, D02_05, D02_06, D03_00, D03_01, D03_02, D03_03, D03_04, D03_05, D03_06, D04_00, D04_01, D04_02, D04_03, D04_04, D04_05, D04_06, D05_00, D05_01, D05_02, D05_03, D05_04, D05_05, D05_06, D06_00, D06_01, D06_02, D06_03, D06_04, D06_05, D06_06, D07_00, D07_01, D07_02, D07_03, D07_04, D07_05, D07_06, D08_00, D08_01, D08_02, D08_03, D08_04, D08_05, D08_06, D09_00, D09_01, D09_02, D09_03, D09_04, D09_05, D09_06: D, random-keyboard-parts:D_SOD-123-Pretty
- removed J0: USB_C_Receptacle_USB2.0, Connector_USB:USB_C_Receptacle_HRO_TYPE-C-31-M-12
- removed JP0: SJ, Jumper:SolderJumper-2_P1.3mm_Open_Pad1.0x1.5mm
- removed LED00_00, LED00_01, LED00_02, LED00_03, LED00_04, LED00_05, LED00_06, LED01_00, LED01_01, LED01_02, LED01_03, LED01_04, LED01_05, LED01_06, LED02_00, LED02_01, LED02_02, LED02_03, LED02_04, LED02_05, LED02_06, LED03_00, LED03_01, LED03_02, LED03_03, LED03_04, LED03_05, LED03_06, LED04_00, LED04_01, LED04_02, LED04_03, LED04_04, LED04_05, LED04_06, LED05_00, LED05_01, LED05_02, LED05_03, LED05_04, LED05_05, LED05_06, LED06_00, LED06_01, LED06_02, LED06_03, LED06_04, LED06_05, LED06_06, LED07_00, LED07_01, LED07_02, LED07_03, LED07_04, LED07_05, LED07_06, LED08_00, LED08_01, LED08_02, LED08_03, LED08_04, LED08_05, LED08_06, LED09_00, LED09_01, LED09_02, LED09_03, LED09_04, LED09_05, LED09_06: SK6812MINI-E, SK6812MINI-E:SK6812MINIE
- removed R0, R1: 22, Resistor_SMD:R_1206_3216Metric
- removed R2, R5, R7, R8: 10k, Resistor_SMD:R_1206_3216Metric
- removed R3, R4: 5.1k, Resistor_SMD:R_1206_3216Metric
- removed R6: 39, Resistor_SMD:R_1206_3216Metric
- removed RESET_SW0: TS-1187A-B-A-B, TS-1187A-B-A-B:SW_TS-1187A-B-A-B
- removed U0: ATmega32U4-A, Package_QFP:TQFP-44_10x10mm_P0.8mm
- removed U1: PMW3360DM-T2QU, PMW3360DM-T2QU:PMW3360
- removed U2: TLV70019DDCR, TLV70019DDCR:Texas_Instruments-TLV70019DDCR-Level_A
- removed U3, U4, U5, U6, U7: 74LVC1T45GW,125, 74LVC1T45GW:Nexperia-SOT363-11_2018-0-IPC_A
- removed Y0: 16Mhz, Crystal:Crystal_SMD_SeikoEpson_FA238-4Pin_3.2x2.5mm
Other:
- board outline removed
