File: case/sandwitch/sandwitch.kicad_pcb (KiCad board)
At the start: 2 copper layers, 339.9 x 106.4 mm, 1 part

Commit message: wip
Other:
- board size 339.9 x 106.4 mm -> 342.9 x 109.6 mm
- board text added: "dynamis v2.0.0 designed by bbrfkr"
- board text removed: "dynamis v1.0.0 designed by bbrfkr"
